File: hardware/pi-adapter-16/pi-adapter.sch (KiCad schematic (older format))
At the start: 32 parts, among them P1 CONN_01X04, P10 CONN_01X04, P11 CONN_01X04, P12 CONN_01X04, P13 CONN_01X04, P14 CONN_01X04, P15 CONN_01X04, P16 CONN_01X04, P2 CONN_01X04, P20 CONN_02X20, P21 I2C, P22 System SPI, P23 UART, P3 CONN_01X04, P30 +5V, P31 GND, P4 CONN_01X04, P5 CONN_01X04, P6 CONN_01X04, P7 CONN_01X04, P8 CONN_01X04, P9 CONN_01X04, U1 74HCT245, U2 74HCT245, U3 74HCT245, U4 74HCT245

Commit message: Prepare for newer KiCAD.
Parts:
- C1, C2, C3, C4: symbol C -> pi-adapter-rescue:C
- C6: symbol C_Small -> pi-adapter-rescue:C_Small
- F1: symbol FUSE -> pi-adapter-rescue:FUSE
- P1, P10, P11, P12, P13, P14, P15, P16, P2, P3, P4, P5, P6, P7, P8, P9: symbol CONN_01X04 -> pi-adapter-rescue:CONN_01X04
- P20: symbol CONN_02X20 -> pi-adapter-rescue:CONN_02X20
- P21, P23: symbol CONN_01X03 -> pi-adapter-rescue:CONN_01X03
- P22: symbol CONN_01X06 -> pi-adapter-rescue:CONN_01X06
- P30, P31: symbol CONN_01X01 -> pi-adapter-rescue:CONN_01X01
- U1, U2, U3, U4: symbol 74HC245 -> pi-adapter-rescue:74HC245
Changed lines of the file:
@@
-EESchema Schematic File Version 2
-LIBS:power
-LIBS:conn
-LIBS:74xx
+EESchema Schematic File Version 4
 LIBS:pi-adapter-cache
-EELAYER 26 0
+EELAYER 29 0
 EELAYER END
 $Descr A4 11693 8268
@@
 $EndDescr
 $Comp
-L 74HC245 U1
+L pi-adapter-rescue:74HC245 U1
 U 1 1 54ECAC85
 P 4550 1750
@@
 $EndComp
 $Comp
-L 74HC245 U2
+L pi-adapter-rescue:74HC245 U2
 U 1 1 54ECB18C
 P 4550 3450
@@
 $EndComp
 $Comp
-L 74HC245 U3
+L pi-adapter-rescue:74HC245 U3
 U 1 1 54ECB1EA
 P 4550 5150
@@
 Connection ~ 2450 2700
 $Comp
-L GND #PWR01
+L pi-adapter-rescue:GND #PWR01
 U 1 1 54ECB417
 P 2500 3600
@@
 	2400 3600 2500 3600
 $Comp
-L GND #PWR02
+L pi-adapter-rescue:GND #PWR02
 U 1 1 54ECB4A1
 P 2500 2900
@@
 	2400 2900 2500 2900
 $Comp
-L GND #PWR03
+L pi-adapter-rescue:GND #PWR03
 U 1 1 54ECB5FE
 P 1800 4600
@@
 	1850 4600 1900 4600
 $Comp
-L GND #PWR04
+L pi-adapter-rescue:GND #PWR04
 U 1 1 54ECB73E
 P 2500 4300
@@
 	2400 4300 2500 4300
 $Comp
-L GND #PWR05
+L pi-adapter-rescue:GND #PWR05
 U 1 1 54ECB7BC
 P 1400 4150
@@
 D5
 $Comp
-L C C1
+L pi-adapter-rescue:C C1
 U 1 1 54ECBE4F
 P 1600 5600
@@
 $EndComp
 $Comp
-L C C2
+L pi-adapter-rescue:C C2
 U 1 1 54ECBEE4
 P 1900 5600
@@
 $EndComp
 $Comp
-L C C3
+L pi-adapter-rescue:C C3
 U 1 1 54ECBF0A
 P 2200 5600
@@
 $EndComp
 $Comp
-L GND #PWR06
+L pi-adapter-rescue:GND #PWR06
 U 1 1 54ECBF56
 P 1900 5850
@@
 Connection ~ 1900 5750
 $Comp
-L VCC #PWR07
+L pi-adapter-rescue:VCC #PWR07
 U 1 1 54ECD0C1
 P 1900 5350
@@
 $EndComp
 $Comp
-L GND #PWR08
+L pi-adapter-rescue:GND #PWR08
 U 1 1 54ECF31C
 P 3850 2300
@@
 	3850 2250 3850 2300
 $Comp
-L GND #PWR09
+L pi-adapter-rescue:GND #PWR09
 U 1 1 54ECF3AB
 P 3850 4000
@@
 $EndComp
 $Comp
-L GND #PWR010
+L pi-adapter-rescue:GND #PWR010
 U 1 1 54ECF608
 P 3850 5700
@@
 clock
 $Comp
-L VCC #PWR011
+L pi-adapter-rescue:VCC #PWR011
 U 1 1 54ED6227
 P 3600 2150
@@
 	3850 2150 3600 2150
 $Comp
-L VCC #PWR012
+L pi-adapter-rescue:VCC #PWR012
 U 1 1 54ED629A
 P 3600 3850
@@
 	3600 3850 3850 3850
 $Comp
-L VCC #PWR013
+L pi-adapter-rescue:VCC #PWR013
 U 1 1 54ED670D
 P 3650 5550
@@
 D1
 $Comp
-L C C4
+L pi-adapter-rescue:C C4
 U 1 1 54F3B6F5
 P 2450 5600
@@
 Connection ~ 2200 5750
 $Comp
-L 74HC245 U4
+L pi-adapter-rescue:74HC245 U4
 U 1 1 54F3F4A2
 P 4550 6950
@@
 $EndComp
 $Comp
-L GND #PWR014
+L pi-adapter-rescue:GND #PWR014
 U 1 1 54F3F4AD
 P 3850 7500
@@
 clock
 $Comp
-L VCC #PWR015
+L pi-adapter-rescue:VCC #PWR015
 U 1 1 54F3F4B9
 P 3650 7350
@@
 NoConn ~ 1900 3500
 $Comp
-L PWR_FLAG #FLG016
+L pi-adapter-rescue:PWR_FLAG #FLG016
 U 1 1 557B23A7
 P 1850 4700
@@
 Connection ~ 1850 4600
 $Comp
-L GND #PWR017
+L pi-adapter-rescue:GND #PWR017
 U 1 1 562B120F
 P 2700 1800
@@
 $EndComp
 $Comp
-L VCC #PWR018
+L pi-adapter-rescue:VCC #PWR018
 U 1 1 562B12CC
 P 1950 1400
@@
 Pi Power 5V
 $Comp
-L C_Small C6
+L pi-adapter-rescue:C_Small C6
 U 1 1 562B2FF4
 P 1300 5600
@@
 $EndComp
 $Comp
-L CONN_01X01 P30
+L pi-adapter-rescue:CONN_01X01 P30
 U 1 1 562B3873
 P 1700 1600
@@
 $EndComp
 $Comp
-L CONN_01X01 P31
+L pi-adapter-rescue:CONN_01X01 P31
 U 1 1 562B38C3
 P 1700 1800
@@
 clock
 $Comp
-L CONN_01X04 P2
+L pi-adapter-rescue:CONN_01X04 P2
 U 1 1 56C16676
 P 5550 1000
@@
 $EndComp
 $Comp
-L CONN_01X04 P1
+L pi-adapter-rescue:CONN_01X04 P1
 U 1 1 56C1694E
 P 5550 2300
@@
 $EndComp
 $Comp
-L CONN_01X04 P10
+L pi-adapter-rescue:CONN_01X04 P10
 U 1 1 56C16C70
 P 6050 1150
@@
 	5250 1850 5600 1850
 $Comp
-L CONN_01X04 P9
+L pi-adapter-rescue:CONN_01X04 P9
 U 1 1 56C17042
 P 6050 2050
@@
 	5900 1700 5900 1850
 $Comp
-L GND #PWR019
+L pi-adapter-rescue:GND #PWR019
 U 1 1 56C176D3
 P 6400 1750
@@
 $EndComp
 $Comp
-L CONN_02X20 P20
+L pi-adapter-rescue:CONN_02X20 P20
 U 1 1 54ECB2B7
 P 2150 3650
@@
 $EndComp
 $Comp
-L CONN_01X03 P23
+L pi-adapter-rescue:CONN_01X03 P23
 U 1 1 56C196A7
 P 3000 3100
@@
 $EndComp
 $Comp
-L GND #PWR020
+L pi-adapter-rescue:GND #PWR020
 U 1 1 56C198BA
 P 2800 3300
@@
 $EndComp
 $Comp
-L CONN_01X03 P21
+L pi-adapter-rescue:CONN_01X03 P21
 U 1 1 56C19AA9
 P 1200 2900
@@
 D16
 $Comp
-L FUSE F1
+L pi-adapter-rescue:FUSE F1
 U 1 1 56C21A23
 P 2250 1600
@@
 Connection ~ 1950 1600
 $Comp
-L VCC #PWR022
+L pi-adapter-rescue:VCC #PWR022
 U 1 1 56C22E4F
 P 2450 2650
@@
 GND CLK DO +5V\n
 $Comp
-L CONN_01X04 P4
+L pi-adapter-rescue:CONN_01X04 P4
 U 1 1 56C22C41
 P 5550 2700
@@
 $EndComp
 $Comp
-L CONN_01X04 P3
+L pi-adapter-rescue:CONN_01X04 P3
 U 1 1 56C22C47
 P 5550 4000
@@
 $EndComp
 $Comp
-L CONN_01X04 P12
+L pi-adapter-rescue:CONN_01X04 P12
 U 1 1 56C22C4D
 P 6050 2850
@@
 	5250 3550 5600 3550
 $Comp
-L CONN_01X04 P11
+L pi-adapter-rescue:CONN_01X04 P11
 U 1 1 56C22C58
 P 6050 3750
@@
 	5900 3400 5900 3550
 $Comp
-L GND #PWR023
+L pi-adapter-rescue:GND #PWR023
 U 1 1 56C22C65
 P 6400 3450
@@
 GND CLK DO +5V\n
 $Comp
-L CONN_01X04 P6
+L pi-adapter-rescue:CONN_01X04 P6
 U 1 1 56C22D24
 P 5550 4400
@@
 $EndComp
 $Comp
-L CONN_01X04 P5
+L pi-adapter-rescue:CONN_01X04 P5
 U 1 1 56C22D2A
 P 5550 5700
@@
 $EndComp
 $Comp
-L CONN_01X04 P14
+L pi-adapter-rescue:CONN_01X04 P14
 U 1 1 56C22D30
 P 6050 4550
@@
 	5250 5250 5600 5250
 $Comp
-L CONN_01X04 P13
+L pi-adapter-rescue:CONN_01X04 P13
 U 1 1 56C22D3B
 P 6050 5450
@@
 	5900 5100 5900 5250
 $Comp
-L GND #PWR024
+L pi-adapter-rescue:GND #PWR024
 U 1 1 56C22D48
 P 6400 5150
@@
 GND CLK DO +5V\n
 $Comp
-L CONN_01X04 P8
+L pi-adapter-rescue:CONN_01X04 P8
 U 1 1 56C22EEF
 P 5550 6200
@@
 $EndComp
 $Comp
-L CONN_01X04 P7
+L pi-adapter-rescue:CONN_01X04 P7
 U 1 1 56C22EF5
 P 5550 7500
@@
 $EndComp
 $Comp
-L CONN_01X04 P16
+L pi-adapter-rescue:CONN_01X04 P16
 U 1 1 56C22EFB
 P 6050 6350
@@
 	5250 7050 5600 7050
 $Comp
-L CONN_01X04 P15
+L pi-adapter-rescue:CONN_01X04 P15
 U 1 1 56C22F06
 P 6050 7250
@@
 	5900 6900 5900 7050
 $Comp
-L GND #PWR025
+L pi-adapter-rescue:GND #PWR025
 U 1 1 56C22F13
 P 6400 6950
@@
 	1400 3800 1900 3800
 $Comp
-L CONN_01X06 P22
+L pi-adapter-rescue:CONN_01X06 P22
 U 1 1 56C265D6
 P 1200 3850
@@
 SCLK
 $Comp
-L PWR_FLAG #FLG026
+L pi-adapter-rescue:PWR_FLAG #FLG026
 U 1 1 56CA81D8
 P 2550 1600
@@
 	1950 1450 1950 1600
 $Comp
-L PWR_FLAG #FLG027
+L pi-adapter-rescue:PWR_FLAG #FLG027
 U 1 1 56CA8545
 P 1950 1450
@@
 	2400 2700 2450 2700
 $Comp
-L GND #PWR028
+L pi-adapter-rescue:GND #PWR028
 U 1 1 56CF0349
 P 2500 4100
@@
 RxD
 $Comp
-L GND #PWR?
+L pi-adapter-rescue:GND #PWR?
 U 1 1 5934A175
 P 1400 3000
