File: hardware/pi-adapter-16/pi-adapter.kicad_pcb (KiCad board)
At the start: 2 copper layers, 64 x 56 mm, 37 parts, among them P1 CONN_01X04, P10 CONN_01X04, P11 CONN_01X04, P12 CONN_01X04, P13 CONN_01X04, P14 CONN_01X04, P15 CONN_01X04, P16 CONN_01X04, P2 CONN_01X04, P20 CONN_02X20, P21 CONN_01X03, P22 CONN_01X06, P23 CONN_01X03, P3 CONN_01X04, P30 +5V, P31 GND, P4 CONN_01X04, P40 CONN_01X01, P41 CONN_01X01, P43 CONN_01X01, P5 CONN_01X04, P6 CONN_01X04, P7 CONN_01X04, P8 CONN_01X04, P9 CONN_01X04, U1 74HCT245, U2 74HCT245, U3 74HCT245, U4 74HCT245

Commit message: Re-save with current kicad 9.x
The last one was done with a 2017-version...
Other:
- net class Default removed
- net class power removed
